Commit message: version out of ros

File: data/neobotixschunk/NeobotixSchunk.urdf (robot description, URDF)
Before this commit: robot gripper_2, 15 links, 14 joints
Links:
- link arm_1_link: geometry collision mesh filename=data/neobotixschunk/meshes/arm_1_link.stl; visual mesh filename=data/neobotixschunk/meshes/arm_1_link.stl
- link arm_2_link: geometry collision mesh filename=data/neobotixschunk/meshes/arm_2_link_collision.stl; visual mesh filename=data/neobotixschunk/meshes/arm_2_link.stl
- link arm_3_link: geometry collision mesh filename=data/neobotixschunk/meshes/arm_3_link_collision.stl; visual mesh filename=data/neobotixschunk/meshes/arm_3_link.stl
- link arm_4_link: geometry collision mesh filename=data/neobotixschunk/meshes/arm_4_link_collision.stl; visual mesh filename=data/neobotixschunk/meshes/arm_4_link.stl
- link arm_5_link: geometry collision mesh filename=data/neobotixschunk/meshes/arm_5_link_collision.stl; visual mesh filename=data/neobotixschunk/meshes/arm_5_link.stl
- link arm_6_link: geometry collision mesh filename=data/neobotixschunk/meshes/arm_6_link_collision.stl; visual mesh filename=data/neobotixschunk/meshes/arm_6_link.stl
- link arm_7_link: geometry collision mesh filename=data/neobotixschunk/meshes/arm_7_link.stl; visual mesh filename=data/neobotixschunk/meshes/arm_7_link.stl
- link arm_podest_link: geometry collision mesh filename=data/neobotixschunk/meshes/arm_podest_link.stl; visual mesh filename=data/neobotixschunk/meshes/arm_podest_link.stl
- link base_link: geometry collision mesh filename=data/neobotixschunk/meshes/MP500-BODY.STL scale=0.01 0.01 0.01; visual mesh filename=data/neobotixschunk/meshes/MP500-BODY.STL scale=0.01 0.01 0.01
- link hanger: geometry collision mesh filename=data/neobotixschunk/meshes/HANGER-WHEEL.STL scale=0.01 0.01 0.01; visual mesh filename=data/neobotixschunk/meshes/HANGER-WHEEL.STL scale=0.01 0.01 0.01
- link laserscanner_front_link: geometry collision cylinder length=0.154 radius=0.053; visual mesh filename=data/neobotixschunk/meshes/SICK-S300.STL
- link wheel_left_link: geometry collision cylinder length=0.085 radius=0.124; visual mesh filename=data/neobotixschunk/meshes/MP500-WHEEL.STL scale=0.01 0.01 0.01
- link wheel_right_link: geometry collision cylinder length=0.085 radius=0.124; visual mesh filename=data/neobotixschunk/meshes/MP500-WHEEL.STL scale=0.01 0.01 0.01

File: data/neobotixschunk/mp500lwa4d.urdf (robot description, URDF)
Before this commit: robot mp500lwa4d_robot, 20 links, 19 joints
Links:
- link arm_1_link: geometry collision mesh filename=data/neobotixschunk/meshes/arm_1_link.stl; visual mesh filename=data/neobotixschunk/meshes/arm_1_link.stl
- link arm_2_link: geometry collision mesh filename=data/neobotixschunk/meshes/arm_2_link_collision.stl; visual mesh filename=data/neobotixschunk/meshes/arm_2_link.stl
- link arm_3_link: geometry collision mesh filename=data/neobotixschunk/meshes/arm_3_link_collision.stl; visual mesh filename=data/neobotixschunk/meshes/arm_3_link.stl
- link arm_4_link: geometry collision mesh filename=data/neobotixschunk/meshes/arm_4_link_collision.stl; visual mesh filename=data/neobotixschunk/meshes/arm_4_link.stl
- link arm_5_link: geometry collision mesh filename=data/neobotixschunk/meshes/arm_5_link_collision.stl; visual mesh filename=data/neobotixschunk/meshes/arm_5_link.stl
- link arm_6_link: geometry collision mesh filename=data/neobotixschunk/meshes/arm_6_link_collision.stl; visual mesh filename=data/neobotixschunk/meshes/arm_6_link.stl
- link arm_7_link: geometry collision mesh filename=data/neobotixschunk/meshes/arm_7_link.stl; visual mesh filename=data/neobotixschunk/meshes/arm_7_link.stl
- link arm_podest_link: geometry collision mesh filename=data/neobotixschunk/meshes/arm_podest_link.stl; visual mesh filename=data/neobotixschunk/meshes/arm_podest_link.stl
- link base_footprint: geometry 
- link base_link: geometry collision mesh filename=data/neobotixschunk/meshes/MP500-BODY.STL scale=0.01 0.01 0.01; visual mesh filename=data/neobotixschunk/meshes/MP500-BODY.STL scale=0.01 0.01 0.01
- link gripper_palm_link: geometry collision box size=0.082 0.114 0.080; visual mesh filename=data/neobotixschunk/meshes/pg70.stl
- link gripper_podest_link: geometry collision mesh filename=data/neobotixschunk/meshes/arm_base_link.stl; visual mesh filename=data/neobotixschunk/meshes/arm_base_link.stl
- link hanger: geometry collision mesh filename=data/neobotixschunk/meshes/HANGER-WHEEL.STL scale=0.01 0.01 0.01; visual mesh filename=data/neobotixschunk/meshes/HANGER-WHEEL.STL scale=0.01 0.01 0.01
- link laserscanner_front_link: geometry collision cylinder length=0.154 radius=0.053; visual mesh filename=data/neobotixschunk/meshes/SICK-S300.STL
- link wheel_left_link: geometry collision cylinder length=0.085 radius=0.125; visual mesh filename=data/neobotixschunk/meshes/MP500-WHEEL.STL scale=0.01 0.01 0.01
- link wheel_right_link: geometry collision cylinder length=0.085 radius=0.125; visual mesh filename=data/neobotixschunk/meshes/MP500-WHEEL.STL scale=0.01 0.01 0.01
