Commit message: neoschunk video fixed

File: data/neobotixschunk/mp500lwa4d_dev.urdf (robot description, URDF)
Before this commit: robot mp500lwa4d_robot, 20 links, 19 joints
Links:
- removed link grasping_frame
- removed link gripper_finger_left_link
- removed link gripper_finger_right_link
- removed link gripper_palm_link
- removed link gripper_podest_link
- removed link laserscanner_front_link
- link base_footprint: mass None -> 0.001
- link base_link: mass 67.010 -> 5; geometry collision box size=0.400 0.676 0.300; visual mesh filename=package://neobotix_schunk_pybullet/data/neobotixschunk/mesh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 scale=0.01 0.01 0.01
- link wheel_left_link: geometry collision cylinder length=0.084 radius=0.125; visual mesh filename=package://neobotix_schunk_pybullet/data/neobotixschunk/mesh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 scale=0.01 0.01 0.01
- link wheel_right_link: geometry collision cylinder length=0.084 radius=0.125; visual mesh filename=package://neobotix_schunk_pybullet/data/neobotixschunk/mesh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 scale=0.01 0.01 0.01
Joints:
- removed joint grasping_frame_joint
- removed joint gripper_finger_left_joint
- removed joint gripper_finger_right_joint
- removed joint gripper_palm_joint
- removed joint gripper_podest_joint
- removed joint laserscanner_front_joint
- joint base_footprint_joint: origin xyz=0 0 0 rpy=0 0 0 -> (none)
- joint wheel_right_joint: limit (none) -> effort=500 velocity=5

File: data/neobotixschunk/mp500lwa4d_devs.urdf (robot description, URDF)
Before this commit: robot mp500lwa4d_robot, 20 links, 19 joints
Links:
- link arm_1_link: geometry collision mesh filename=package://mp500lwa4d_description/meshes/lwa4d/arm_1_link.stl; visual mesh filename=package://mp500lwa4d_description/meshes/lwa4d/arm_1_link.stl
- link arm_2_link: geometry collision mesh filename=package://mp500lwa4d_description/meshes/lwa4d/arm_2_link_co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; visual mesh filename=package://mp500lwa4d_description/meshes/lwa4d/arm_2_link.stl
- link arm_3_link: geometry collision mesh filename=package://mp500lwa4d_description/meshes/lwa4d/arm_3_link_co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; visual mesh filename=package://mp500lwa4d_description/meshes/lwa4d/arm_3_link.stl
- link arm_4_link: geometry collision mesh filename=package://mp500lwa4d_description/meshes/lwa4d/arm_4_link_co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; visual mesh filename=package://mp500lwa4d_description/meshes/lwa4d/arm_4_link.stl
- link arm_5_link: geometry collision mesh filename=package://mp500lwa4d_description/meshes/lwa4d/arm_5_link_co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; visual mesh filename=package://mp500lwa4d_description/meshes/lwa4d/arm_5_link.stl
- link arm_6_link: geometry collision mesh filename=package://mp500lwa4d_description/meshes/lwa4d/arm_6_link_co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; visual mesh filename=package://mp500lwa4d_description/meshes/lwa4d/arm_6_link.stl
- link arm_7_link: geometry collision mesh filename=package://mp500lwa4d_description/meshes/lwa4d/arm_7_link.stl scale=0.9 0.9 0.9; visual mesh filename=package://mp500lwa4d_description/meshes/lwa4d/arm_7_link.stl
- link arm_podest_link: geometry collision mesh filename=package://mp500lwa4d_description/meshes/lwa4d/arm_podest_li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; visual mesh filename=package://mp500lwa4d_description/meshes/lwa4d/arm_podest_li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
- link base_footprint: mass None -> 0.0001
- link base_link: mass 67.010 -> 15; geometry collision box size=0.585 0.676 0.300; visual mesh filename=package://mp500lwa4d_description/meshes/mp500/MP500-BODY.STL scale=0.01 0.01 0.01
- link grasping_frame: mass None -> 0.0001
- link gripper_finger_left_link: mass 0.01 -> 0.001
- link gripper_finger_right_link: mass 0.01 -> 0.001
- link gripper_palm_link: mass 0.01 -> 0.001; geometry collision box size=0.082 0.114 0.080; visual mesh filename=package://mp500lwa4d_description/meshes/pg70/pg70.dae
- link gripper_podest_link: geometry collision mesh filename=package://mp500lwa4d_description/meshes/pg70/arm_base_link.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; visual mesh filename=package://mp500lwa4d_description/meshes/pg70/arm_base_link.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
- link hanger: mass 0.01 -> 1; geometry collision sphere radius=0.125; visual mesh filename=package://mp500lwa4d_description/meshes/mp500/HANGER-WHEEL.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 scale=0.01 0.01 0.01
- link laserscanner_front_link: geometry collision cylinder length=0.154 radius=0.053; visual mesh filename=package://mp500lwa4d_description/meshes/mp500/SICK-S300.STL
- link wheel_left_link: mass 1.5 -> 1; geometry collision cylinder length=0.085 radius=0.125; visual mesh filename=package://mp500lwa4d_description/meshes/mp500/MP500-WHEEL.S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 scale=0.01 0.01 0.01
- link wheel_right_link: mass 1.5 -> 1; geometry collision cylinder length=0.085 radius=0.125; visual mesh filename=package://mp500lwa4d_description/meshes/mp500/MP500-WHEEL.S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 scale=0.01 0.01 0.01
Joints:
- joint arm_6_joint: origin xyz=0 0 0.323 rpy=-1.57079632679 -1.57079632679 0 -> xyz=0.00 0.00 0.323 rpy=-1.57079632679 -1.57079632679 0
- joint arm_7_joint: origin xyz=0 0 0 rpy=1.57079632679 0 1.57079632679 -> xyz=0.00 0 0 rpy=1.57079632679 0 1.57079632679
- joint base_footprint_joint: origin xyz=0 0 0 rpy=0 0 0 -> (none)
- joint hanger_joint: origin xyz=0.255 0 0.11 rpy=0 0 0 -> xyz=0.255 0 0.125 rpy=0 0 0
- joint wheel_left_joint: origin xyz=-0.155 0.255 0.13 rpy=0 0 0 -> xyz=-0.155 0.255 0.125 rpy=0 0 0
- joint wheel_right_joint: limit (none) -> effort=500 velocity=5; origin xyz=-0.155 -0.255 0.13 rpy=0 0 0 -> xyz=-0.155 -0.255 0.125 rpy=0 0 0

File: data/plane.urdf (robot description, URDF)
Before this commit: robot plane, 1 links, 0 joints
Links:
- removed link planeLink
- added link planelink, mass .0; collision box size=30 30 10; visual mesh filename=plane.obj scale=1 1 1

File: data/spheregoal.urdf (robot description, URDF)
Before this commit: robot urdf_robot, 1 links, 0 joints
Links:
- removed link base_link
- added link spherelink, mass 0.0; visual sphere radius=0.03
