Commit message: add ik

File: data/neobotixschunk/arm_lwa4d.urdf (robot description, URDF)
Before this commit: robot arm_lwa4d, 9 links, 8 joints
Links:
- added link gripper_podest_link, mass 0.01
- link arm_podest_link: mass 1 -> 0.01
Joints:
- added joint gripper_podest_joint: type fixed, parent arm_7_link, child gripper_podest_link, origin xyz=0 0 0.0824 rpy=0 0 0

File: data/neobotixschunk/base_mp500.urdf (robot description, URDF)
Before this commit: robot base_mp500, 5 links, 4 joints
Links:
- link base_footprint: mass None -> 0.0001; geometry 
- link base_link: mass 1 -> 15; geometry collision box size=0.585 0.676 0.300; visual mesh filename=package://mp500lwa4d_description/meshes/mp500/MP500-BODY.STL scale=0.01 0.01 0.01
- link hanger: mass 0.01 -> 1
Joints:
- joint hanger_joint: origin xyz=0.255 0 0.11 rpy=0 0 0 -> xyz=0.255 0 0.125 rpy=0 0 0
- joint wheel_left_joint: origin xyz=-0.155 0.255 0.13 rpy=0 0 0 -> xyz=-0.155 0.255 0.125 rpy=0 0 0
- joint wheel_right_joint: origin xyz=-0.155 -0.255 0.13 rpy=0 0 0 -> xyz=-0.155 -0.255 0.125 rpy=0 0 0

File: data/neobotixschunk/mp500lwa4d.urdf (robot description, URDF)
Before this commit: robot mp500lwa4d_robot, 20 links, 19 joints
Links:
- link arm_6_link: geometry collision mesh filename=package://neobotix_schunk_pybullet/data/neobotixschunk/mesh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 scale=0.9 0.9 0.9; visual mesh filename=package://neobotix_schunk_pybullet/data/neobotixschunk/mesh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
- link gripper_finger_left_link: geometry collision box size=0.03 0.005 0.08; visual box size=0.03 0.01 0.08
- link gripper_finger_right_link: geometry collision box size=0.03 0.005 0.08; visual box size=0.03 0.01 0.08
Joints:
- joint gripper_finger_left_joint: limit lower=-0.0301 upper=-0.005 effort=10 velocity=0.041 -> lower=-0.0301 upper=-0.01 effort=10 velocity=0.041; type prismatic -> fixed
- joint gripper_finger_right_joint: limit lower=0.005 upper=0.0301 effort=10 velocity=0.041 -> lower=0.01 upper=0.0301 effort=10 velocity=0.041; type prismatic -> fixed
