Commit message: modified from megi

File: data/neobotixschunk/mp500lwa4d.urdf (robot description, URDF)
Before this commit: robot mp500lwa4d_robot, 20 links, 19 joints
Links:
- link gripper_finger_left_link: mass 0.00 -> 0.01
- link gripper_finger_right_link: mass 0.00 -> 0.01
- link gripper_palm_link: mass 0.001 -> 0.01
- link gripper_podest_link: mass 0.001 -> 0.01

Commit message: path fised

File: data/neobotixschunk/mp500lwa4d.urdf (robot description, URDF)
Before this commit: robot mp500lwa4d_robot, 20 links, 19 joints
Links:
- link arm_7_link: geometry collision mesh filename=package://neobotix_schunk_pybullet/data/neobotixschunk/mesh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 scale=0.9 0.9 0.9; visual mesh filename=package://neobotix_schunk_pybullet/data/neobotixschunk/mesh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
- link base_footprint: mass None -> 0.0001
- link base_link: mass 67.010 -> 15; geometry collision box size=0.585 0.676 0.300; visual mesh filename=package://neobotix_schunk_pybullet/data/neobotixschunk/mesh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 scale=0.01 0.01 0.01
- link grasping_frame: mass None -> 0.0001
- link gripper_finger_left_link: mass 0.01 -> 0.001
- link gripper_finger_right_link: mass 0.01 -> 0.001
- link gripper_palm_link: mass 0.01 -> 0.001
- link hanger: mass 0.01 -> 1; geometry collision sphere radius=0.125; visual mesh filename=package://neobotix_schunk_pybullet/data/neobotixschunk/mesh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 scale=0.01 0.01 0.01
- link wheel_left_link: mass 1.5 -> 1
- link wheel_right_link: mass 1.5 -> 1
Joints:
- joint arm_6_joint: origin xyz=0 0 0.323 rpy=-1.57079632679 -1.57079632679 0 -> xyz=0.00 0.00 0.323 rpy=-1.57079632679 -1.57079632679 0
- joint arm_7_joint: origin xyz=0 0 0 rpy=1.57079632679 0 1.57079632679 -> xyz=0.00 0 0 rpy=1.57079632679 0 1.57079632679
- joint base_footprint_joint: origin xyz=0 0 0 rpy=0 0 0 -> (none)
- joint hanger_joint: origin xyz=0.255 0 0.11 rpy=0 0 0 -> xyz=0.255 0 0.125 rpy=0 0 0
- joint wheel_left_joint: origin xyz=-0.155 0.255 0.13 rpy=0 0 0 -> xyz=-0.155 0.255 0.125 rpy=0 0 0
- joint wheel_right_joint: limit (none) -> effort=500 velocity=5; origin xyz=-0.155 -0.255 0.13 rpy=0 0 0 -> xyz=-0.155 -0.255 0.125 rpy=0 0 0

Commit message: reset

File: data/neobotixschunk/mp500lwa4d.urdf (robot description, URDF)
Before this commit: robot mp500lwa4d_robot, 20 links, 19 joints
Joints:
- joint gripper_finger_left_joint: origin xyz=0 -0.005 0.1139 rpy=0 0 0 -> xyz=0 -0.025 0.1139 rpy=0 0 0
- joint gripper_finger_right_joint: origin xyz=0 0.005 0.1139 rpy=-0 0 0 -> xyz=0 0.025 0.1139 rpy=-0 0 0
